File: Hardware/MAST.kicad_pcb (KiCad board)
At the start: 6 copper layers, 26 x 15 mm, 122 parts, among them J1 S+, J2 S-, J3 S-, J4 BAT+, J5 BAT-, Q1 DMP21D0UFB4, Q2 PMZ290UNE2, U1 LP5907SNX-3.0, U2 TPS62748, U3 ARTIC-R2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

Commit message: Increase silkscreen text size & removed some text
Other:
- board text removed: "3V3"
- board text removed: "CLK"
- board text removed: "DIO"
- board text removed: "EN"
- board text removed: "GND"
- board text removed: "MISO"
- board text removed: "MOSI"
- board text removed: "RST"
